Commit message: Moved pa10 7a meshes to add pa10 7c meshes Fixed pa10a to use its own mesh and its own macro name Added pa10c xacro Adapted launch files and xacros to use this new robot

File: pa10-c.urdf.xacro (robot description, xacro)
@@ -1,4 +1,4 @@
 <?xml version="1.0"?>
-<robot name="PA10a"
+<robot name="PA10c"
 		 xmlns:xacro="http://www.ros.org/wiki/xacro"
 		 xmlns:sensor="http://playerstage.sourceforge.net/gazebo/xmlschema/#sensor"
@@ -6,10 +6,10 @@
        xmlns:interface="http://playerstage.sourceforge.net/gazebo/xmlschema/#interface">
   <xacro:include filename="$(find agni_description)/urdf/util.urdf.xacro"/>
-  <macro name="pa10a_arm" params="name">
+  <macro name="pa10c_arm" params="name">
   <link name="${name}arm_base_link">
     <visual>
       <origin xyz="0 0 0" rpy="0 0 0"/>
       <geometry>
-        <mesh filename="package://agni_description/pa10/meshes/pa-7a/link0_mesh.dae" scale="1 1 1" />
+        <mesh filename="package://agni_description/pa10/meshes/pa-7c/link0_mesh.dae" scale="1 1 1" />
       </geometry>
     </visual>
@@ -17,5 +17,5 @@
       <origin xyz="0 0 0.115" rpy="0 0 0"/>
       <geometry>
-		  <cylinder length="0.23" radius="0.112"/>
+		  <cylinder length="0.200" radius="0.112"/>
       </geometry>
     </collision>
@@ -30,11 +30,11 @@
       <origin xyz="0 0 0" rpy="0 0 0"/>
       <geometry>
-        <mesh filename="package://agni_description/pa10/meshes/pa-7a/link1_mesh.dae" scale="1 1 1" />
-      </geometry>
-    </visual>
-    <collision>
-      <origin xyz="0 0 0" rpy="0 0 0"/>
-      <geometry>
-        <mesh filename="package://agni_description/pa10/meshes/pa-7a/link1_mesh.dae" scale="1 1 1" />
+        <mesh filename="package://agni_description/pa10/meshes/pa-7c/link1_mesh.dae" scale="1 1 1" />
+      </geometry>
+    </visual>
+    <collision>
+      <origin xyz="0 0 0" rpy="0 0 0"/>
+      <geometry>
+        <mesh filename="package://agni_description/pa10/meshes/pa-7c/link1_mesh.dae" scale="1 1 1" />
       </geometry>
     </collision>
@@ -47,13 +47,13 @@
   <link name="${name}arm_2_link">
     <visual>
-      <origin xyz="0 0 -0.315" rpy="0 0 0"/>
-      <geometry>
-        <mesh filename="package://agni_description/pa10/meshes/pa-7a/link2_mesh.dae" scale="1 1 1" />
-      </geometry>
-    </visual>
-    <collision>
-      <origin xyz="0 0 -0.315" rpy="0 0 0"/>
-      <geometry>
-        <mesh filename="package://agni_description/pa10/meshes/pa-7a/link2_mesh.dae" scale="1 1 1" />
+      <origin xyz="0 0 -0.317" rpy="0 0 0"/>
+      <geometry>
+        <mesh filename="package://agni_description/pa10/meshes/pa-7c/link2_mesh.dae" scale="1 1 1" />
+      </geometry>
+    </visual>
+    <collision>
+      <origin xyz="0 0 -0.317" rpy="0 0 0"/>
+      <geometry>
+        <mesh filename="package://agni_description/pa10/meshes/pa-7c/link2_mesh.dae" scale="1 1 1" />
       </geometry>
     </collision>
@@ -66,13 +66,13 @@
   <link name="${name}arm_3_link">
     <visual>
-      <origin xyz="0 0 -0.315" rpy="0 0 0"/>
-      <geometry>
-        <mesh filename="package://agni_description/pa10/meshes/pa-7a/link3_mesh.dae" scale="1 1 1" />
-      </geometry>
-    </visual>
-    <collision>
-      <origin xyz="0 0 -0.315" rpy="0 0 0"/>
-      <geometry>
-        <mesh filename="package://agni_description/pa10/meshes/pa-7a/link3_mesh.dae" scale="1 1 1" />
+      <origin xyz="0 0 -0.317" rpy="0 0 0"/>
+      <geometry>
+        <mesh filename="package://agni_description/pa10/meshes/pa-7c/link3_mesh.dae" scale="1 1 1" />
+      </geometry>
+    </visual>
+    <collision>
+      <origin xyz="0 0 -0.317" rpy="0 0 0"/>
+      <geometry>
+        <mesh filename="package://agni_description/pa10/meshes/pa-7c/link3_mesh.dae" scale="1 1 1" />
       </geometry>
     </collision>
@@ -85,13 +85,13 @@
   <link name="${name}arm_4_link">
     <visual>
-      <origin xyz="0 0 -0.765" rpy="0 0 0"/>
-      <geometry>
-        <mesh filename="package://agni_description/pa10/meshes/pa-7a/link4_mesh.dae" scale="1 1 1" />
-      </geometry>
-    </visual>
-    <collision>
-      <origin xyz="0 0 -0.765" rpy="0 0 0"/>
-      <geometry>
-        <mesh filename="package://agni_description/pa10/meshes/pa-7a/link4_mesh.dae" scale="1 1 1" />
+      <origin xyz="0 0 -0.767" rpy="0 0 0"/>
+      <geometry>
+        <mesh filename="package://agni_description/pa10/meshes/pa-7c/link4_mesh.dae" scale="1 1 1" />
+      </geometry>
+    </visual>
+    <collision>
+      <origin xyz="0 0 -0.767" rpy="0 0 0"/>
+      <geometry>
+        <mesh filename="package://agni_description/pa10/meshes/pa-7c/link4_mesh.dae" scale="1 1 1" />
       </geometry>
     </collision>
@@ -104,13 +104,13 @@
   <link name="${name}arm_5_link">
     <visual>
-      <origin xyz="0 0 -0.765" rpy="0 0 0"/>
-      <geometry>
-        <mesh filename="package://agni_description/pa10/meshes/pa-7a/link5_mesh.dae" scale="1 1 1" />
-      </geometry>
-    </visual>
-    <collision>
-      <origin xyz="0 0 -0.765" rpy="0 0 0"/>
-      <geometry>
-        <mesh filename="package://agni_description/pa10/meshes/pa-7a/link5_mesh.dae" scale="1 1 1" />
+      <origin xyz="0 0 -0.767" rpy="0 0 0"/>
+      <geometry>
+        <mesh filename="package://agni_description/pa10/meshes/pa-7c/link5_mesh.dae" scale="1 1 1" />
+      </geometry>
+    </visual>
+    <collision>
+      <origin xyz="0 0 -0.767" rpy="0 0 0"/>
+      <geometry>
+        <mesh filename="package://agni_description/pa10/meshes/pa-7c/link5_mesh.dae" scale="1 1 1" />
       </geometry>
     </collision>
@@ -123,13 +123,13 @@
   <link name="${name}arm_6_link">
     <visual>
-      <origin xyz="0 0 -1.265" rpy="0 0 0"/>
-      <geometry>
-        <mesh filename="package://agni_description/pa10/meshes/pa-7a/link6_mesh.dae" scale="1 1 1" />
-      </geometry>
-    </visual>
-    <collision>
-      <origin xyz="0 0 -1.265" rpy="0 0 0"/>
-      <geometry>
-        <mesh filename="package://agni_description/pa10/meshes/pa-7a/link6_mesh.dae" scale="1 1 1" />
+      <origin xyz="0 0 -1.247" rpy="0 0 0"/>
+      <geometry>
+        <mesh filename="package://agni_description/pa10/meshes/pa-7c/link6_mesh.dae" scale="1 1 1" />
+      </geometry>
+    </visual>
+    <collision>
+      <origin xyz="0 0 -1.247" rpy="0 0 0"/>
+      <geometry>
+        <mesh filename="package://agni_description/pa10/meshes/pa-7c/link6_mesh.dae" scale="1 1 1" />
       </geometry>
     </collision>
@@ -142,18 +142,18 @@
   <link name="${name}arm_7_link">
     <visual>
-      <origin xyz="0 0 1.35" rpy="0 0 0"/>
-      <geometry>
-        <mesh filename="package://agni_description/pa10/meshes/pa-7a/link7_mesh.dae" scale="1 1 1" />
-      </geometry>
-    </visual>
-    <collision>
-      <origin xyz="0 0 1.345" rpy="0 0 0"/>
-      <geometry>
-        <mesh filename="package://agni_description/pa10/meshes/pa-7a/link7_mesh.dae" scale="1 1 1" />
-      </geometry>
-    </collision>
-    <inertial>
-      <mass value="1" />
-      <origin xyz="0 0 2.22045e-16" rpy="0 0 0"/>
+      <origin xyz="0 0 1.317" rpy="0 0 0"/>
+      <geometry>
+        <mesh filename="package://agni_description/pa10/meshes/pa-7c/link7_mesh.dae" scale="1 1 1" />
+      </geometry>
+    </visual>
+    <collision>
+      <origin xyz="0 0 1.317" rpy="0 0 0"/>
+      <geometry>
+        <mesh filename="package://agni_description/pa10/meshes/pa-7c/link7_mesh.dae" scale="1 1 1" />
+      </geometry>
+    </collision>
+    <inertial>
+      <mass value="1" />
+      <origin xyz="0 0 0" rpy="0 0 0"/>
       <inertia ixx="1" ixy="0" ixz="0" iyy="1" iyz="0" izz="1"/>
     </inertial>
@@ -164,5 +164,5 @@
     <origin xyz="0 0 0" rpy="0 0 0 "/>
     <axis   xyz="0 0 1"/>
-    <limit lower="${-177/180*M_PI}" upper="${177/180*M_PI}" effort="100000" velocity="0.5" />
+    <limit lower="${-177/180*M_PI}" upper="${177/180*M_PI}" effort="100" velocity="0.5" />
     <dynamics damping="0.2" friction="0" />
   </joint>
@@ -170,7 +170,7 @@
     <parent link="${name}arm_1_link"/>
     <child  link="${name}arm_2_link"/>
-    <origin xyz="0 0 0.315" rpy="0 0 0 "/>
+    <origin xyz="0 0 0.317" rpy="0 0 0 "/>
     <axis   xyz="0 1 0"/>
-    <limit lower="${-94/180*M_PI}" upper="${+94/180*M_PI}" effort="100000" velocity="0.5" />
+    <limit lower="${-94/180*M_PI}" upper="${+94/180*M_PI}" effort="100" velocity="0.5" />
     <dynamics damping="0.2" friction="0" />
   </joint>
@@ -180,5 +180,5 @@
     <origin xyz="0 0 0" rpy="0 0 0 "/>
     <axis   xyz="0 0 1"/>
-    <limit lower="${-174/180*M_PI}" upper="${174/180*M_PI}" effort="100000" velocity="0.5" />
+    <limit lower="${-174/180*M_PI}" upper="${174/180*M_PI}" effort="100" velocity="0.5" />
     <dynamics damping="0.2" friction="0" />
   </joint>
@@ -188,5 +188,5 @@
     <origin xyz="0 0 0.45" rpy="0 0 0 "/>
     <axis   xyz="0 1 0"/>
-    <limit lower="${-137/180*M_PI}" upper="${137/180*M_PI}" effort="100000" velocity="0.5" />
+    <limit lower="${-137/180*M_PI}" upper="${137/180*M_PI}" effort="100" velocity="0.5" />
     <dynamics damping="0.2" friction="0" />
   </joint>
@@ -196,5 +196,5 @@
     <origin xyz="0 0 0" rpy="0 0 0 "/>
     <axis   xyz="0 0 1"/>
-    <limit lower="${-255/180*M_PI}" upper="${255/180*M_PI}" effort="100000" velocity="0.5" />
+    <limit lower="${-255/180*M_PI}" upper="${255/180*M_PI}" effort="100" velocity="0.5" />
     <dynamics damping="0.2" friction="0" />
   </joint>
@@ -202,7 +202,7 @@
     <parent link="${name}arm_5_link"/>
     <child  link="${name}arm_6_link"/>
-    <origin xyz="0 0 0.5" rpy="0 0 0 "/>
+    <origin xyz="0 0 0.480" rpy="0 0 0 "/>
     <axis   xyz="0 1 0"/>
-    <limit lower="${-100/180*M_PI}" upper="${100/180*M_PI}" effort="100000" velocity="0.5" />
+    <limit lower="${-165/180*M_PI}" upper="${165/180*M_PI}" effort="100" velocity="0.5" />
     <dynamics damping="0.2" friction="0" />
   </joint>
@@ -210,7 +210,7 @@
     <parent link="${name}arm_6_link"/>
     <child  link="${name}arm_7_link"/>
-    <origin xyz="0 0 0.08" rpy="0 0 0 "/>
-    <axis   xyz="0 0 1"/>
-    <limit lower="${-255/180*M_PI}" upper="${255/180*M_PI}" effort="100000" velocity="0.5" />
+    <origin xyz="0 0 0.07" rpy="0 0 0 "/>
+    <axis   xyz="0 0 1"/>
+    <limit lower="${-255/180*M_PI}" upper="${255/180*M_PI}" effort="100" velocity="0.5" />
     <dynamics damping="0.2" friction="0" />
   </joint>
