Commit message: Changed pa10 colors and fixed meshes (decimate + position) Corrected kinematic parameters

File: pa10-a.urdf.xacro (robot description, xacro)
@@ -142,5 +142,5 @@
   <link name="${name}arm_7_link">
     <visual>
-      <origin xyz="0 0 1.35" rpy="0 0 0"/>
+      <origin xyz="0 0 1.345" rpy="0 0 0"/>
       <geometry>
         <mesh filename="package://agni_description/pa10/meshes/pa-7a/link7_mesh.dae" scale="1 1 1" />
@@ -164,5 +164,5 @@
     <origin xyz="0 0 0" rpy="0 0 0 "/>
     <axis   xyz="0 0 1"/>
-    <limit lower="${-177/180*M_PI}" upper="${177/180*M_PI}" effort="100000" velocity="0.5" />
+    <limit lower="${-177/180*M_PI}" upper="${177/180*M_PI}" effort="100" velocity="1" />
     <dynamics damping="0.2" friction="0" />
   </joint>
@@ -172,5 +172,5 @@
     <origin xyz="0 0 0.315" rpy="0 0 0 "/>
     <axis   xyz="0 1 0"/>
-    <limit lower="${-94/180*M_PI}" upper="${+94/180*M_PI}" effort="100000" velocity="0.5" />
+    <limit lower="${-91/180*M_PI}" upper="${+91/180*M_PI}" effort="100" velocity="1" />
     <dynamics damping="0.2" friction="0" />
   </joint>
@@ -180,5 +180,5 @@
     <origin xyz="0 0 0" rpy="0 0 0 "/>
     <axis   xyz="0 0 1"/>
-    <limit lower="${-174/180*M_PI}" upper="${174/180*M_PI}" effort="100000" velocity="0.5" />
+    <limit lower="${-174/180*M_PI}" upper="${174/180*M_PI}" effort="100" velocity="2" />
     <dynamics damping="0.2" friction="0" />
   </joint>
@@ -188,5 +188,5 @@
     <origin xyz="0 0 0.45" rpy="0 0 0 "/>
     <axis   xyz="0 1 0"/>
-    <limit lower="${-137/180*M_PI}" upper="${137/180*M_PI}" effort="100000" velocity="0.5" />
+    <limit lower="${-137/180*M_PI}" upper="${137/180*M_PI}" effort="100" velocity="2" />
     <dynamics damping="0.2" friction="0" />
   </joint>
@@ -196,5 +196,5 @@
     <origin xyz="0 0 0" rpy="0 0 0 "/>
     <axis   xyz="0 0 1"/>
-    <limit lower="${-255/180*M_PI}" upper="${255/180*M_PI}" effort="100000" velocity="0.5" />
+    <limit lower="${-255/180*M_PI}" upper="${255/180*M_PI}" effort="100" velocity="6.28" />
     <dynamics damping="0.2" friction="0" />
   </joint>
@@ -204,5 +204,5 @@
     <origin xyz="0 0 0.5" rpy="0 0 0 "/>
     <axis   xyz="0 1 0"/>
-    <limit lower="${-100/180*M_PI}" upper="${100/180*M_PI}" effort="100000" velocity="0.5" />
+    <limit lower="${-165/180*M_PI}" upper="${165/180*M_PI}" effort="100" velocity="6.28" />
     <dynamics damping="0.2" friction="0" />
   </joint>
@@ -212,5 +212,5 @@
     <origin xyz="0 0 0.08" rpy="0 0 0 "/>
     <axis   xyz="0 0 1"/>
-    <limit lower="${-255/180*M_PI}" upper="${255/180*M_PI}" effort="100000" velocity="0.5" />
+    <limit lower="${-359/180*M_PI}" upper="${359/180*M_PI}" effort="100" velocity="6.28" />
     <dynamics damping="0.2" friction="0" />
   </joint>

File: pa10-c.urdf.xacro (robot description, xacro)
@@ -142,5 +142,5 @@
   <link name="${name}arm_7_link">
     <visual>
-      <origin xyz="0 0 1.317" rpy="0 0 0"/>
+      <origin xyz="0 0 0" rpy="0 0 0"/>
       <geometry>
         <mesh filename="package://agni_description/pa10/meshes/pa-7c/link7_mesh.dae" scale="1 1 1" />
@@ -148,5 +148,5 @@
     </visual>
     <collision>
-      <origin xyz="0 0 1.317" rpy="0 0 0"/>
+      <origin xyz="0 0 0" rpy="0 0 0"/>
       <geometry>
         <mesh filename="package://agni_description/pa10/meshes/pa-7c/link7_mesh.dae" scale="1 1 1" />
@@ -164,5 +164,5 @@
     <origin xyz="0 0 0" rpy="0 0 0 "/>
     <axis   xyz="0 0 1"/>
-    <limit lower="${-177/180*M_PI}" upper="${177/180*M_PI}" effort="100" velocity="0.5" />
+    <limit lower="${-177/180*M_PI}" upper="${177/180*M_PI}" effort="100" velocity="1" />
     <dynamics damping="0.2" friction="0" />
   </joint>
@@ -172,5 +172,5 @@
     <origin xyz="0 0 0.317" rpy="0 0 0 "/>
     <axis   xyz="0 1 0"/>
-    <limit lower="${-94/180*M_PI}" upper="${+94/180*M_PI}" effort="100" velocity="0.5" />
+    <limit lower="${-94/180*M_PI}" upper="${+94/180*M_PI}" effort="100" velocity="1" />
     <dynamics damping="0.2" friction="0" />
   </joint>
@@ -180,5 +180,5 @@
     <origin xyz="0 0 0" rpy="0 0 0 "/>
     <axis   xyz="0 0 1"/>
-    <limit lower="${-174/180*M_PI}" upper="${174/180*M_PI}" effort="100" velocity="0.5" />
+    <limit lower="${-174/180*M_PI}" upper="${174/180*M_PI}" effort="100" velocity="2" />
     <dynamics damping="0.2" friction="0" />
   </joint>
@@ -188,5 +188,5 @@
     <origin xyz="0 0 0.45" rpy="0 0 0 "/>
     <axis   xyz="0 1 0"/>
-    <limit lower="${-137/180*M_PI}" upper="${137/180*M_PI}" effort="100" velocity="0.5" />
+    <limit lower="${-137/180*M_PI}" upper="${137/180*M_PI}" effort="100" velocity="2" />
     <dynamics damping="0.2" friction="0" />
   </joint>
@@ -196,5 +196,5 @@
     <origin xyz="0 0 0" rpy="0 0 0 "/>
     <axis   xyz="0 0 1"/>
-    <limit lower="${-255/180*M_PI}" upper="${255/180*M_PI}" effort="100" velocity="0.5" />
+    <limit lower="${-255/180*M_PI}" upper="${255/180*M_PI}" effort="100" velocity="6.28" />
     <dynamics damping="0.2" friction="0" />
   </joint>
@@ -204,5 +204,5 @@
     <origin xyz="0 0 0.480" rpy="0 0 0 "/>
     <axis   xyz="0 1 0"/>
-    <limit lower="${-165/180*M_PI}" upper="${165/180*M_PI}" effort="100" velocity="0.5" />
+    <limit lower="${-165/180*M_PI}" upper="${165/180*M_PI}" effort="100" velocity="6.28" />
     <dynamics damping="0.2" friction="0" />
   </joint>
@@ -212,5 +212,5 @@
     <origin xyz="0 0 0.07" rpy="0 0 0 "/>
     <axis   xyz="0 0 1"/>
-    <limit lower="${-255/180*M_PI}" upper="${255/180*M_PI}" effort="100" velocity="0.5" />
+    <limit lower="${-255/180*M_PI}" upper="${255/180*M_PI}" effort="100" velocity="6.28" />
     <dynamics damping="0.2" friction="0" />
   </joint>
