Commit message: Set pa10 correct masses according to mitsubishi documentation and quite good inertia estimation Changed pa10 collision models to sets of primitives

File: pa10-a.urdf.xacro (robot description, xacro)
@@ -15,18 +15,24 @@
     </visual>
     <collision>
-      <origin xyz="0 0 0.115" rpy="0 0 0"/>
-      <geometry>
-		  <cylinder length="0.23" radius="0.112"/>
-      </geometry>
-    </collision>
-    <inertial>
-      <mass value="1" />
+      <origin xyz="0 0 0.100" rpy="0 0 0"/>
+      <geometry>
+		  <cylinder length="0.20" radius="0.115"/>
+      </geometry>
+    </collision>
+    <collision>
+       <origin xyz="0 0.120 0.060" rpy="0 0 0"/>
+      <geometry>
+        <box size="0.130 0.060 0.060" />
+      </geometry>
+    </collision>
+    <inertial>
+      <mass value="3.04" />
+      <origin xyz="0 0 0.075" rpy="0 0 0"/>
+      <inertia ixx="0.0193" ixy="0" ixz="0" iyy="0.0193" iyz="0" izz="0.0184"/>
+    </inertial>
+  </link>
+  <link name="${name}arm_1_link">
+    <visual>
       <origin xyz="0 0 0" rpy="0 0 0"/>
-      <inertia ixx="1" ixy="0" ixz="0" iyy="1" iyz="0" izz="1"/>
-    </inertial>
-  </link>
-  <link name="${name}arm_1_link">
-    <visual>
-      <origin xyz="0 0 0" rpy="0 0 0"/>
       <geometry>
         <mesh filename="package://agni_description/pa10/meshes/pa-7a/link1_mesh.dae" scale="1 1 1" />
@@ -34,13 +40,25 @@
     </visual>
     <collision>
-      <origin xyz="0 0 0" rpy="0 0 0"/>
-      <geometry>
-        <mesh filename="package://agni_description/pa10/meshes/pa-7a/link1_mesh.dae" scale="1 1 1" />
-      </geometry>
-    </collision>
-    <inertial>
-      <mass value="1" />
-      <origin xyz="0 0 0" rpy="0 0 0"/>
-      <inertia ixx="1" ixy="0" ixz="0" iyy="1" iyz="0" izz="1"/>
+      <origin xyz="0 0 0.210" rpy="0 0 0"/>
+      <geometry>
+        <cylinder length="0.020" radius="0.110"/>
+      </geometry>
+    </collision>
+    <collision>
+      <origin xyz="0.0 0.104 0.298" rpy="0 0 0"/>
+      <geometry>
+		  <box size="0.140 0.05 0.180" />
+      </geometry>
+    </collision>
+    <collision>
+      <origin xyz="0.0 -0.104 0.298" rpy="0 0 0"/>
+      <geometry>
+		  <box size="0.140 0.05 0.180" />
+      </geometry>
+    </collision>
+    <inertial>
+      <mass value="9.78" />
+      <origin xyz="0 0 0.148" rpy="0 0 0"/>
+      <inertia ixx="0.145" ixy="0" ixz="0" iyy="0.145" iyz="0" izz="0.049"/>
     </inertial>
   </link>
@@ -53,32 +71,50 @@
     </visual>
     <collision>
+      <origin xyz="0 0 0.181" rpy="0 0 0"/>
+      <geometry>
+        <cylinder length="0.266" radius="0.07"/>
+      </geometry>
+    </collision>
+    <collision>
+      <origin xyz="0 0 0.0" rpy="1.5708 0 0"/>
+      <geometry>
+        <cylinder length="0.160" radius="0.075"/>
+      </geometry>
+    </collision>
+    <inertial>
+      <mass value="8.41" />
+      <origin xyz="0 0 0.06325" rpy="0 0 0"/>
+      <inertia ixx="0.1316" ixy="0" ixz="0" iyy="0.1316" iyz="0" izz="0.0206"/>
+    </inertial>
+  </link>
+  <link name="${name}arm_3_link">
+    <visual>
       <origin xyz="0 0 -0.315" rpy="0 0 0"/>
       <geometry>
-        <mesh filename="package://agni_description/pa10/meshes/pa-7a/link2_mesh.dae" scale="1 1 1" />
-      </geometry>
-    </collision>
-    <inertial>
-      <mass value="1" />
-      <origin xyz="0 0 0" rpy="0 0 0"/>
-      <inertia ixx="1" ixy="0" ixz="0" iyy="1" iyz="0" izz="1"/>
-    </inertial>
-  </link>
-  <link name="${name}arm_3_link">
-    <visual>
-      <origin xyz="0 0 -0.315" rpy="0 0 0"/>
-      <geometry>
         <mesh filename="package://agni_description/pa10/meshes/pa-7a/link3_mesh.dae" scale="1 1 1" />
       </geometry>
     </visual>
     <collision>
-      <origin xyz="0 0 -0.315" rpy="0 0 0"/>
-      <geometry>
-        <mesh filename="package://agni_description/pa10/meshes/pa-7a/link3_mesh.dae" scale="1 1 1" />
-      </geometry>
-    </collision>
-    <inertial>
-      <mass value="1" />
-      <origin xyz="0 0 0" rpy="0 0 0"/>
-      <inertia ixx="1" ixy="0" ixz="0" iyy="1" iyz="0" izz="1"/>
+      <origin xyz="0 0 0.336" rpy="0 0 0"/>
+      <geometry>
+         <box size="0.120 0.116 0.044" />
+      </geometry>
+    </collision>
+    <collision>
+      <origin xyz="0.0 0.083 0.411" rpy="0 0 0"/>
+      <geometry>
+		  <box size="0.120 0.05 0.20" />
+      </geometry>
+    </collision>
+    <collision>
+      <origin xyz="0.0 -0.083 0.411" rpy="0 0 0"/>
+      <geometry>
+		  <box size="0.120 0.05 0.20" />
+      </geometry>
+    </collision>
+    <inertial>
+      <mass value="3.51" />
+      <origin xyz="0 0 0.3605" rpy="0 0 0"/>
+      <inertia ixx="0.0298" ixy="0" ixz="0" iyy="0.0298" iyz="0" izz="0.009"/>
     </inertial>
   </link>
@@ -91,32 +127,50 @@
     </visual>
     <collision>
+      <origin xyz="0 0 0.150" rpy="0 0 0"/>
+      <geometry>
+        <cylinder length="0.248" radius="0.055"/>
+      </geometry>
+    </collision>
+    <collision>
+      <origin xyz="0 0 0.0" rpy="1.5708 0 0"/>
+      <geometry>
+        <cylinder length="0.116" radius="0.055"/>
+      </geometry>
+    </collision>
+    <inertial>
+      <mass value="4.31" />
+      <origin xyz="0 0 0.04609" rpy="0 0 0"/>
+      <inertia ixx="0.0493" ixy="0" ixz="0" iyy="0.0493" iyz="0" izz="0.0065"/>
+    </inertial>
+  </link>
+  <link name="${name}arm_5_link">
+    <visual>
       <origin xyz="0 0 -0.765" rpy="0 0 0"/>
       <geometry>
-        <mesh filename="package://agni_description/pa10/meshes/pa-7a/link4_mesh.dae" scale="1 1 1" />
-      </geometry>
-    </collision>
-    <inertial>
-      <mass value="1" />
-      <origin xyz="0 0 0" rpy="0 0 0"/>
-      <inertia ixx="1" ixy="0" ixz="0" iyy="1" iyz="0" izz="1"/>
-    </inertial>
-  </link>
-  <link name="${name}arm_5_link">
-    <visual>
-      <origin xyz="0 0 -0.765" rpy="0 0 0"/>
-      <geometry>
         <mesh filename="package://agni_description/pa10/meshes/pa-7a/link5_mesh.dae" scale="1 1 1" />
       </geometry>
     </visual>
     <collision>
-      <origin xyz="0 0 -0.765" rpy="0 0 0"/>
-      <geometry>
-        <mesh filename="package://agni_description/pa10/meshes/pa-7a/link5_mesh.dae" scale="1 1 1" />
-      </geometry>
-    </collision>
-    <inertial>
-      <mass value="1" />
-      <origin xyz="0 0 0" rpy="0 0 0"/>
-      <inertia ixx="1" ixy="0" ixz="0" iyy="1" iyz="0" izz="1"/>
+      <origin xyz="0 0 0.300" rpy="0 0 0"/>
+      <geometry>
+         <box size="0.09 0.082 0.070" />
+      </geometry>
+    </collision>
+    <collision>
+      <origin xyz="0.0 0.051 0.401" rpy="0 0 0"/>
+      <geometry>
+		  <box size="0.09 0.03 0.284" />
+      </geometry>
+    </collision>
+    <collision>
+      <origin xyz="0.0 -0.051 0.401" rpy="0 0 0"/>
+      <geometry>
+		  <box size="0.09 0.03 0.284" />
+      </geometry>
+    </collision>
+    <inertial>
+      <mass value="3.45" />
+      <origin xyz="0 0 0.335" rpy="0 0 0"/>
+      <inertia ixx="0.0486" ixy="0" ixz="0" iyy="0.0486" iyz="0" izz="0.0052"/>
     </inertial>
   </link>
@@ -129,13 +183,13 @@
     </visual>
     <collision>
-      <origin xyz="0 0 -1.265" rpy="0 0 0"/>
-      <geometry>
-        <mesh filename="package://agni_description/pa10/meshes/pa-7a/link6_mesh.dae" scale="1 1 1" />
-      </geometry>
-    </collision>
-    <inertial>
-      <mass value="1" />
-      <origin xyz="0 0 0" rpy="0 0 0"/>
-      <inertia ixx="1" ixy="0" ixz="0" iyy="1" iyz="0" izz="1"/>
+      <origin xyz="0 0 -0.045" rpy="0 0 0"/>
+      <geometry>
+        <cylinder length="0.228" radius="0.045"/>
+      </geometry>
+    </collision>
+    <inertial>
+      <mass value="1.46" />
+      <origin xyz="0 0 -0.03" rpy="0 0 0"/>
+      <inertia ixx="0.0071" ixy="0" ixz="0" iyy="0.0071" iyz="0" izz="0.0015"/>
     </inertial>
   </link>
@@ -148,13 +202,13 @@
     </visual>
     <collision>
-      <origin xyz="0 0 1.345" rpy="0 0 0"/>
-      <geometry>
-        <mesh filename="package://agni_description/pa10/meshes/pa-7a/link7_mesh.dae" scale="1 1 1" />
-      </geometry>
-    </collision>
-    <inertial>
-      <mass value="1" />
-      <origin xyz="0 0 2.22045e-16" rpy="0 0 0"/>
-      <inertia ixx="1" ixy="0" ixz="0" iyy="1" iyz="0" izz="1"/>
+      <origin xyz="0 0 -0.01" rpy="0 0 0"/>
+      <geometry>
+        <cylinder length="0.02" radius="0.04"/>
+      </geometry>
+    </collision>
+    <inertial>
+      <mass value="0.24" />
+      <origin xyz="0 0 -0.029" rpy="0 0 0"/>
+      <inertia ixx="0.0001" ixy="0" ixz="0" iyy="0.0001" iyz="0" izz="0.0002"/>
     </inertial>
   </link>

File: pa10-c.urdf.xacro (robot description, xacro)
@@ -15,146 +15,200 @@
     </visual>
     <collision>
-      <origin xyz="0 0 0.115" rpy="0 0 0"/>
-      <geometry>
-		  <cylinder length="0.200" radius="0.112"/>
-      </geometry>
-    </collision>
-    <inertial>
-      <mass value="1" />
+      <origin xyz="0 0 0.100" rpy="0 0 0"/>
+      <geometry>
+        <cylinder length="0.200" radius="0.115"/>
+      </geometry>
+    </collision>
+    <collision>
+      <origin xyz="0 0.130 0.090" rpy="0 0 0"/>
+      <geometry>
+        <box size="0.160 0.080 0.160" />
+      </geometry>
+    </collision>
+    <inertial>
+      <mass value="6.88" />
+      <origin xyz="0 0 0.091" rpy="0 0 0"/>
+      <inertia ixx="0.043" ixy="0" ixz="0" iyy="0.043" iyz="0" izz="0.0416"/>
+    </inertial>
+  </link>
+  <link name="${name}arm_1_link">
+    <visual>
       <origin xyz="0 0 0" rpy="0 0 0"/>
-      <inertia ixx="1" ixy="0" ixz="0" iyy="1" iyz="0" izz="1"/>
-    </inertial>
-  </link>
-  <link name="${name}arm_1_link">
+      <geometry>
+        <mesh filename="package://agni_description/pa10/meshes/pa-7c/link1_mesh.dae" scale="1 1 1" />
+      </geometry>
+    </visual>
+    <collision>
+      <origin xyz="0 0 0.210" rpy="0 0 0"/>
+      <geometry>
+        <cylinder length="0.020" radius="0.110"/>
+      </geometry>
+    </collision>
+    <collision>
+      <origin xyz="0.0 0.105 0.3" rpy="0 0 0"/>
+      <geometry>
+		  <box size="0.140 0.05 0.180" />
+      </geometry>
+    </collision>
+    <collision>
+      <origin xyz="0.0 -0.105 0.3" rpy="0 0 0"/>
+      <geometry>
+		  <box size="0.140 0.05 0.180" />
+      </geometry>
+    </collision>
+    <inertial>
+      <mass value="7.33" />
+      <origin xyz="0 0 0.160" rpy="0 0 0"/>
+      <inertia ixx="0.11" ixy="0" ixz="0" iyy="0.11" iyz="0" izz="0.037"/>
+    </inertial>
+  </link>
+  <link name="${name}arm_2_link">
+    <visual>
+      <origin xyz="0 0 -0.317" rpy="0 0 0"/>
+      <geometry>
+        <mesh filename="package://agni_description/pa10/meshes/pa-7c/link2_mesh.dae" scale="1 1 1" />
+      </geometry>
+    </visual>
+    <collision>
+      <origin xyz="0 0 0.183" rpy="0 0 0"/>
+      <geometry>
+        <cylinder length="0.266" radius="0.07"/>
+      </geometry>
+    </collision>
+    <collision>
+      <origin xyz="0 0 0.0" rpy="1.5708 0 0"/>
+      <geometry>
+        <cylinder length="0.160" radius="0.075"/>
+      </geometry>
+    </collision>
+    <inertial>
+      <mass value="10.76" />
+      <origin xyz="0 0 0.063" rpy="0 0 0"/>
+      <inertia ixx="0.168" ixy="0" ixz="0" iyy="0.168" iyz="0" izz="0.026"/>
+    </inertial>
+  </link>
+  <link name="${name}arm_3_link">
+    <visual>
+      <origin xyz="0 0 -0.317" rpy="0 0 0"/>
+      <geometry>
+        <mesh filename="package://agni_description/pa10/meshes/pa-7c/link3_mesh.dae" scale="1 1 1" />
+      </geometry>
+    </visual>
+    <collision>
+      <origin xyz="0 0 0.333" rpy="0 0 0"/>
+      <geometry>
+         <box size="0.120 0.116 0.034" />
+      </geometry>
+    </collision>
+    <collision>
+      <origin xyz="0.0 0.083 0.413" rpy="0 0 0"/>
+      <geometry>
+		  <box size="0.120 0.05 0.20" />
+      </geometry>
+    </collision>
+    <collision>
+      <origin xyz="0.0 -0.083 0.413" rpy="0 0 0"/>
+      <geometry>
+		  <box size="0.120 0.05 0.20" />
+      </geometry>
+    </collision>
+    <inertial>
+      <mass value="2.97" />
+      <origin xyz="0 0 0.346" rpy="0 0 0"/>
+      <inertia ixx="0.028" ixy="0" ixz="0" iyy="0.028" iyz="0" izz="0.073"/>
+    </inertial>
+  </link>
+  <link name="${name}arm_4_link">
+    <visual>
+      <origin xyz="0 0 -0.767" rpy="0 0 0"/>
+      <geometry>
+        <mesh filename="package://agni_description/pa10/meshes/pa-7c/link4_mesh.dae" scale="1 1 1" />
+      </geometry>
+    </visual>
+    <collision>
+      <origin xyz="0 0 0.170" rpy="0 0 0"/>
+      <geometry>
+        <cylinder length="0.248" radius="0.055"/>
+      </geometry>
+    </collision>
+    <collision>
+      <origin xyz="0 0 0.0" rpy="1.5708 0 0"/>
+      <geometry>
+        <cylinder length="0.116" radius="0.055"/>
+      </geometry>
+    </collision>
+    <inertial>
+      <mass value="4.86" />
+      <origin xyz="0 0 0.0485" rpy="0 0 0"/>
+      <inertia ixx="0.0055" ixy="0" ixz="0" iyy="0.0055" iyz="0" izz="0.0073"/>
+    </inertial>
+  </link>
+  <link name="${name}arm_5_link">
+    <visual>
+      <origin xyz="0 0 -0.767" rpy="0 0 0"/>
+      <geometry>
+        <mesh filename="package://agni_description/pa10/meshes/pa-7c/link5_mesh.dae" scale="1 1 1" />
+      </geometry>
+    </visual>
+    <collision>
+      <origin xyz="0 0 0.322" rpy="0 0 0"/>
+      <geometry>
+         <box size="0.09 0.102 0.070" />
+      </geometry>
+    </collision>
+    <collision>
+      <origin xyz="0.0 0.066 0.403" rpy="0 0 0"/>
+      <geometry>
+		  <box size="0.09 0.03 0.242" />
+      </geometry>
+    </collision>
+    <collision>
+      <origin xyz="0.0 -0.066 0.403" rpy="0 0 0"/>
+      <geometry>
+		  <box size="0.09 0.03 0.242" />
+      </geometry>
+    </collision>
+    <inertial>
+      <mass value="3.08" />
+      <origin xyz="0 0 0.368" rpy="0 0 0"/>
+      <inertia ixx="0.02" ixy="0" ixz="0" iyy="0.02" iyz="0" izz="0.0046"/>
+    </inertial>
+  </link>
+  <link name="${name}arm_6_link">
+    <visual>
+      <origin xyz="0 0 -1.247" rpy="0 0 0"/>
+      <geometry>
+        <mesh filename="package://agni_description/pa10/meshes/pa-7c/link6_mesh.dae" scale="1 1 1" />
+      </geometry>
+    </visual>
+    <collision>
+      <origin xyz="0 0 -0.023" rpy="0 0 0"/>
+      <geometry>
+        <cylinder length="0.186" radius="0.05"/>
+      </geometry>
+    </collision>
+    <inertial>
+      <mass value="3.00" />
+      <origin xyz="0 0 -0.042" rpy="0 0 0"/>
+      <inertia ixx="0.011" ixy="0" ixz="0" iyy="0.011" iyz="0" izz="0.0038"/>
+    </inertial>
+  </link>
+  <link name="${name}arm_7_link">
     <visual>
       <origin xyz="0 0 0" rpy="0 0 0"/>
       <geometry>
-        <mesh filename="package://agni_description/pa10/meshes/pa-7c/link1_mesh.dae" scale="1 1 1" />
-      </geometry>
-    </visual>
-    <collision>
-      <origin xyz="0 0 0" rpy="0 0 0"/>
-      <geometry>
-        <mesh filename="package://agni_description/pa10/meshes/pa-7c/link1_mesh.dae" scale="1 1 1" />
-      </geometry>
-    </collision>
-    <inertial>
-      <mass value="1" />
-      <origin xyz="0 0 0" rpy="0 0 0"/>
-      <inertia ixx="1" ixy="0" ixz="0" iyy="1" iyz="0" izz="1"/>
-    </inertial>
-  </link>
-  <link name="${name}arm_2_link">
-    <visual>
-      <origin xyz="0 0 -0.317" rpy="0 0 0"/>
-      <geometry>
-        <mesh filename="package://agni_description/pa10/meshes/pa-7c/link2_mesh.dae" scale="1 1 1" />
-      </geometry>
-    </visual>
-    <collision>
-      <origin xyz="0 0 -0.317" rpy="0 0 0"/>
-      <geometry>
-        <mesh filename="package://agni_description/pa10/meshes/pa-7c/link2_mesh.dae" scale="1 1 1" />
-      </geometry>
-    </collision>
-    <inertial>
-      <mass value="1" />
-      <origin xyz="0 0 0" rpy="0 0 0"/>
-      <inertia ixx="1" ixy="0" ixz="0" iyy="1" iyz="0" izz="1"/>
-    </inertial>
-  </link>
-  <link name="${name}arm_3_link">
-    <visual>
-      <origin xyz="0 0 -0.317" rpy="0 0 0"/>
-      <geometry>
-        <mesh filename="package://agni_description/pa10/meshes/pa-7c/link3_mesh.dae" scale="1 1 1" />
-      </geometry>
-    </visual>
-    <collision>
-      <origin xyz="0 0 -0.317" rpy="0 0 0"/>
-      <geometry>
-        <mesh filename="package://agni_description/pa10/meshes/pa-7c/link3_mesh.dae" scale="1 1 1" />
-      </geometry>
-    </collision>
-    <inertial>
-      <mass value="1" />
-      <origin xyz="0 0 0" rpy="0 0 0"/>
-      <inertia ixx="1" ixy="0" ixz="0" iyy="1" iyz="0" izz="1"/>
-    </inertial>
-  </link>
-  <link name="${name}arm_4_link">
-    <visual>
-      <origin xyz="0 0 -0.767" rpy="0 0 0"/>
-      <geometry>
-        <mesh filename="package://agni_description/pa10/meshes/pa-7c/link4_mesh.dae" scale="1 1 1" />
-      </geometry>
-    </visual>
-    <collision>
-      <origin xyz="0 0 -0.767" rpy="0 0 0"/>
-      <geometry>
-        <mesh filename="package://agni_description/pa10/meshes/pa-7c/link4_mesh.dae" scale="1 1 1" />
-      </geometry>
-    </collision>
-    <inertial>
-      <mass value="1" />
-      <origin xyz="0 0 0" rpy="0 0 0"/>
-      <inertia ixx="1" ixy="0" ixz="0" iyy="1" iyz="0" izz="1"/>
-    </inertial>
-  </link>
-  <link name="${name}arm_5_link">
-    <visual>
-      <origin xyz="0 0 -0.767" rpy="0 0 0"/>
-      <geometry>
-        <mesh filename="package://agni_description/pa10/meshes/pa-7c/link5_mesh.dae" scale="1 1 1" />
-      </geometry>
-    </visual>
-    <collision>
-      <origin xyz="0 0 -0.767" rpy="0 0 0"/>
-      <geometry>
-        <mesh filename="package://agni_description/pa10/meshes/pa-7c/link5_mesh.dae" scale="1 1 1" />
-      </geometry>
-    </collision>
-    <inertial>
-      <mass value="1" />
-      <origin xyz="0 0 0" rpy="0 0 0"/>
-      <inertia ixx="1" ixy="0" ixz="0" iyy="1" iyz="0" izz="1"/>
-    </inertial>
-  </link>
-  <link name="${name}arm_6_link">
-    <visual>
-      <origin xyz="0 0 -1.247" rpy="0 0 0"/>
-      <geometry>
-        <mesh filename="package://agni_description/pa10/meshes/pa-7c/link6_mesh.dae" scale="1 1 1" />
-      </geometry>
-    </visual>
-    <collision>
-      <origin xyz="0 0 -1.247" rpy="0 0 0"/>
-      <geometry>
-        <mesh filename="package://agni_description/pa10/meshes/pa-7c/link6_mesh.dae" scale="1 1 1" />
-      </geometry>
-    </collision>
-    <inertial>
-      <mass value="1" />
-      <origin xyz="0 0 0" rpy="0 0 0"/>
-      <inertia ixx="1" ixy="0" ixz="0" iyy="1" iyz="0" izz="1"/>
-    </inertial>
-  </link>
-  <link name="${name}arm_7_link">
-    <visual>
-      <origin xyz="0 0 0" rpy="0 0 0"/>
-      <geometry>
         <mesh filename="package://agni_description/pa10/meshes/pa-7c/link7_mesh.dae" scale="1 1 1" />
       </geometry>
     </visual>
     <collision>
-      <origin xyz="0 0 0" rpy="0 0 0"/>
-      <geometry>
-        <mesh filename="package://agni_description/pa10/meshes/pa-7c/link7_mesh.dae" scale="1 1 1" />
-      </geometry>
-    </collision>
-    <inertial>
-      <mass value="1" />
-      <origin xyz="0 0 0" rpy="0 0 0"/>
-      <inertia ixx="1" ixy="0" ixz="0" iyy="1" iyz="0" izz="1"/>
+      <origin xyz="0 0 -0.01" rpy="0 0 0"/>
+      <geometry>
+        <cylinder length="0.02" radius="0.04"/>
+      </geometry>
+    </collision>
+    <inertial>
+      <mass value="0.12" />
+      <origin xyz="0 0 -0.048" rpy="0 0 0"/>
+      <inertia ixx="0.000052" ixy="0.0" ixz="0" iyy="0.000052" iyz="0" izz="0.000096"/>
     </inertial>
   </link>
