Commit message: Added controllers in pa10 (shadow version due to prob in ros_control) Added args to set the gazebo default arm posture (not working yet) Fixed pa10a urdf (forearm rotated 180 deg)

File: pa10-a.urdf.xacro (robot description, xacro)
@@ -32,4 +32,8 @@
     </inertial>
   </link>
+  <gazebo reference="${name}arm_base_link">
+    <material>LightGrey</material>
+    <selfCollide>false</selfCollide>
+  </gazebo>
   <link name="${name}arm_1_link">
     <visual>
@@ -65,5 +69,5 @@
   <link name="${name}arm_2_link">
     <visual>
-      <origin xyz="0 0 -0.315" rpy="0 0 0"/>
+      <origin xyz="0 0 -0.315" rpy="0 0 3.1415"/>
       <geometry>
         <mesh filename="package://agni_description/pa10/meshes/pa-7a/link2_mesh.dae" scale="1 1 1" />
@@ -221,4 +225,9 @@
     <dynamics damping="0.2" friction="0" />
   </joint>
+  <transmission type="sr_mechanism_model/SimpleTransmission" name="${name}S1_transmission">
+    <actuator name="${name}S1_actuator" />
+    <joint name="${name}S1">
+    </joint>
+  </transmission>
   <joint name="${name}S2" type="revolute">
     <parent link="${name}arm_1_link"/>
@@ -229,4 +238,9 @@
     <dynamics damping="0.2" friction="0" />
   </joint>
+  <transmission type="sr_mechanism_model/SimpleTransmission" name="${name}S2_transmission">
+    <actuator name="${name}S2_actuator" />
+    <joint name="${name}S2">
+    </joint>
+  </transmission>
   <joint name="${name}S3" type="revolute">
     <parent link="${name}arm_2_link"/>
@@ -237,4 +251,9 @@
     <dynamics damping="0.2" friction="0" />
   </joint>
+  <transmission type="sr_mechanism_model/SimpleTransmission" name="${name}S3_transmission">
+    <actuator name="${name}S3_actuator" />
+    <joint name="${name}S3">
+    </joint>
+  </transmission>
   <joint name="${name}E1" type="revolute">
     <parent link="${name}arm_3_link"/>
@@ -245,4 +264,9 @@
     <dynamics damping="0.2" friction="0" />
   </joint>
+  <transmission type="sr_mechanism_model/SimpleTransmission" name="${name}E1_transmission">
+    <actuator name="${name}E1_actuator" />
+    <joint name="${name}E1">
+    </joint>
+  </transmission>
   <joint name="${name}E2" type="revolute">
     <parent link="${name}arm_4_link"/>
@@ -253,4 +277,9 @@
     <dynamics damping="0.2" friction="0" />
   </joint>
+  <transmission type="sr_mechanism_model/SimpleTransmission" name="${name}E2_transmission">
+    <actuator name="${name}E2_actuator" />
+    <joint name="${name}E2">
+    </joint>
+  </transmission>
   <joint name="${name}W1" type="revolute">
     <parent link="${name}arm_5_link"/>
@@ -261,4 +290,10 @@
     <dynamics damping="0.2" friction="0" />
   </joint>
+  <!-- <transmission type="transmission_interface/SimpleTransmission" name="${name}W1_transmission"> -->
+  <transmission type="sr_mechanism_model/SimpleTransmission" name="${name}W1_transmission">
+    <actuator name="${name}W1_actuator" />
+    <joint name="${name}W1">
+    </joint>
+  </transmission>
   <joint name="${name}W2" type="revolute">
     <parent link="${name}arm_6_link"/>
@@ -269,4 +304,9 @@
     <dynamics damping="0.2" friction="0" />
   </joint>
+  <transmission type="sr_mechanism_model/SimpleTransmission" name="${name}W2_transmission">
+    <actuator name="${name}W2_actuator" />
+    <joint name="${name}W2">
+    </joint>
+  </transmission>
   <joint name="${name}arm_hand_fixed_joint" type="fixed">
 	 <parent link="${name}arm_7_link"/>

File: pa10-c.urdf.xacro (robot description, xacro)
@@ -32,4 +32,8 @@
     </inertial>
   </link>
+  <gazebo reference="${name}arm_base_link">
+    <material>LightGrey</material>
+    <selfCollide>false</selfCollide>
+  </gazebo>
   <link name="${name}arm_1_link">
     <visual>
@@ -221,4 +225,9 @@
     <dynamics damping="0.2" friction="0" />
   </joint>
+  <transmission type="sr_mechanism_model/SimpleTransmission" name="${name}S1_transmission">
+    <actuator name="${name}S1_actuator" />
+    <joint name="${name}S1">
+    </joint>
+  </transmission>
   <joint name="${name}S2" type="revolute">
     <parent link="${name}arm_1_link"/>
@@ -229,4 +238,9 @@
     <dynamics damping="0.2" friction="0" />
   </joint>
+  <transmission type="sr_mechanism_model/SimpleTransmission" name="${name}S2_transmission">
+    <actuator name="${name}S2_actuator" />
+    <joint name="${name}S2">
+    </joint>
+  </transmission>
   <joint name="${name}S3" type="revolute">
     <parent link="${name}arm_2_link"/>
@@ -237,4 +251,9 @@
     <dynamics damping="0.2" friction="0" />
   </joint>
+  <transmission type="sr_mechanism_model/SimpleTransmission" name="${name}S3_transmission">
+    <actuator name="${name}S3_actuator" />
+    <joint name="${name}S3">
+    </joint>
+  </transmission>
   <joint name="${name}E1" type="revolute">
     <parent link="${name}arm_3_link"/>
@@ -245,4 +264,9 @@
     <dynamics damping="0.2" friction="0" />
   </joint>
+  <transmission type="sr_mechanism_model/SimpleTransmission" name="${name}E1_transmission">
+    <actuator name="${name}E1_actuator" />
+    <joint name="${name}E1">
+    </joint>
+  </transmission>
   <joint name="${name}E2" type="revolute">
     <parent link="${name}arm_4_link"/>
@@ -253,4 +277,9 @@
     <dynamics damping="0.2" friction="0" />
   </joint>
+  <transmission type="sr_mechanism_model/SimpleTransmission" name="${name}E2_transmission">
+    <actuator name="${name}E2_actuator" />
+    <joint name="${name}E2">
+    </joint>
+  </transmission>
   <joint name="${name}W1" type="revolute">
     <parent link="${name}arm_5_link"/>
@@ -261,4 +290,10 @@
     <dynamics damping="0.2" friction="0" />
   </joint>
+  <!-- <transmission type="transmission_interface/SimpleTransmission" name="${name}W1_transmission"> -->
+  <transmission type="sr_mechanism_model/SimpleTransmission" name="${name}W1_transmission">
+    <actuator name="${name}W1_actuator" />
+    <joint name="${name}W1">
+    </joint>
+  </transmission>
   <joint name="${name}W2" type="revolute">
     <parent link="${name}arm_6_link"/>
@@ -269,4 +304,9 @@
     <dynamics damping="0.2" friction="0" />
   </joint>
+  <transmission type="sr_mechanism_model/SimpleTransmission" name="${name}W2_transmission">
+    <actuator name="${name}W2_actuator" />
+    <joint name="${name}W2">
+    </joint>
+  </transmission>
   <joint name="${name}arm_hand_fixed_joint" type="fixed">
 	 <parent link="${name}arm_7_link"/>

Commit message: Fixed urdf to remove self-collisions between link 5 and 7 on pa10-a

File: pa10-a.urdf.xacro (robot description, xacro)
@@ -187,7 +187,7 @@
     </visual>
     <collision>
-      <origin xyz="0 0 -0.045" rpy="0 0 0"/>
-      <geometry>
-        <cylinder length="0.228" radius="0.045"/>
+      <origin xyz="0 0 -0.043" rpy="0 0 0"/>
+      <geometry>
+        <cylinder length="0.230" radius="0.035"/>
       </geometry>
     </collision>
@@ -208,5 +208,5 @@
       <origin xyz="0 0 -0.01" rpy="0 0 0"/>
       <geometry>
-        <cylinder length="0.02" radius="0.04"/>
+        <cylinder length="0.02" radius="0.035"/>
       </geometry>
     </collision>

Commit message: added missing xacro: prefixes

File: pa10-a.urdf.xacro (robot description, xacro)
@@ -6,5 +6,5 @@
        xmlns:interface="http://playerstage.sourceforge.net/gazebo/xmlschema/#interface">
   <xacro:include filename="$(find agni_description)/urdf/util.urdf.xacro"/>
-  <macro name="pa10a_arm" params="name kinematic:=false">
+  <xacro:macro name="pa10a_arm" params="name kinematic:=false">
   <link name="${name}arm_base_link">
     <visual>
@@ -367,4 +367,4 @@
     <kinematic>${kinematic}</kinematic>
   </gazebo>
-  </macro>
+  </xacro:macro>
 </robot>

File: pa10-c.urdf.xacro (robot description, xacro)
@@ -6,5 +6,5 @@
        xmlns:interface="http://playerstage.sourceforge.net/gazebo/xmlschema/#interface">
   <xacro:include filename="$(find agni_description)/urdf/util.urdf.xacro"/>
-  <macro name="pa10c_arm" params="name kinematic:=false">
+  <xacro:macro name="pa10c_arm" params="name kinematic:=false">
   <link name="${name}arm_base_link">
     <visual>
@@ -367,4 +367,4 @@
     <kinematic>${kinematic}</kinematic>
   </gazebo>
-  </macro>
+  </xacro:macro>
 </robot>

File: pa10_shadow_controller_manager.xacro (robot description, xacro)
@@ -5,5 +5,5 @@
        xmlns:interface="http://playerstage.sourceforge.net/gazebo/xmlschema/#interface">
 	<!-- namespace must be set up according to launch file namespace -->
-  <macro name="pa10_shadow_gazebo_controller_manager" params="namespace">
+  <xacro:macro name="pa10_shadow_gazebo_controller_manager" params="namespace">
 		<gazebo>
 			<plugin name="sr_gazebo_ros_controller_manager" filename="libsr_gazebo_ros_controller_manager.so">
@@ -13,4 +13,4 @@
 			</plugin>
 		</gazebo>
-  </macro>
+  </xacro:macro>
 </robot>

Commit message: replace M_PI with pi

File: pa10-a.urdf.xacro (robot description, xacro)
@@ -244,5 +244,5 @@
     <origin xyz="0 0 0" rpy="0 0 0 "/>
     <axis   xyz="0 0 1"/>
-    <limit lower="${-177/180*M_PI}" upper="${177/180*M_PI}" effort="100" velocity="1" />
+    <limit lower="${-177/180*pi}" upper="${177/180*pi}" effort="100" velocity="1" />
     <dynamics damping="0.2" friction="0" />
   </joint>
@@ -261,5 +261,5 @@
     <origin xyz="0 0 0.315" rpy="0 0 0 "/>
     <axis   xyz="0 1 0"/>
-    <limit lower="${-91/180*M_PI}" upper="${+91/180*M_PI}" effort="100" velocity="1" />
+    <limit lower="${-91/180*pi}" upper="${+91/180*pi}" effort="100" velocity="1" />
     <dynamics damping="0.2" friction="0" />
   </joint>
@@ -278,5 +278,5 @@
     <origin xyz="0 0 0" rpy="0 0 0 "/>
     <axis   xyz="0 0 1"/>
-    <limit lower="${-174/180*M_PI}" upper="${174/180*M_PI}" effort="100" velocity="2" />
+    <limit lower="${-174/180*pi}" upper="${174/180*pi}" effort="100" velocity="2" />
     <dynamics damping="0.2" friction="0" />
   </joint>
@@ -295,5 +295,5 @@
     <origin xyz="0 0 0.45" rpy="0 0 0 "/>
     <axis   xyz="0 1 0"/>
-    <limit lower="${-137/180*M_PI}" upper="${137/180*M_PI}" effort="100" velocity="2" />
+    <limit lower="${-137/180*pi}" upper="${137/180*pi}" effort="100" velocity="2" />
     <dynamics damping="0.2" friction="0" />
   </joint>
@@ -312,5 +312,5 @@
     <origin xyz="0 0 0" rpy="0 0 0 "/>
     <axis   xyz="0 0 1"/>
-    <limit lower="${-255/180*M_PI}" upper="${255/180*M_PI}" effort="100" velocity="6.28" />
+    <limit lower="${-255/180*pi}" upper="${255/180*pi}" effort="100" velocity="6.28" />
     <dynamics damping="0.2" friction="0" />
   </joint>
@@ -329,5 +329,5 @@
     <origin xyz="0 0 0.5" rpy="0 0 0 "/>
     <axis   xyz="0 1 0"/>
-    <limit lower="${-165/180*M_PI}" upper="${165/180*M_PI}" effort="100" velocity="6.28" />
+    <limit lower="${-165/180*pi}" upper="${165/180*pi}" effort="100" velocity="6.28" />
     <dynamics damping="0.2" friction="0" />
   </joint>
@@ -347,5 +347,5 @@
     <origin xyz="0 0 0.08" rpy="0 0 0 "/>
     <axis   xyz="0 0 1"/>
-    <limit lower="${-359/180*M_PI}" upper="${359/180*M_PI}" effort="100" velocity="6.28" />
+    <limit lower="${-359/180*pi}" upper="${359/180*pi}" effort="100" velocity="6.28" />
     <dynamics damping="0.2" friction="0" />
   </joint>

File: pa10-c.urdf.xacro (robot description, xacro)
@@ -244,5 +244,5 @@
     <origin xyz="0 0 0" rpy="0 0 0 "/>
     <axis   xyz="0 0 1"/>
-    <limit lower="${-177/180*M_PI}" upper="${177/180*M_PI}" effort="100" velocity="1" />
+    <limit lower="${-177/180*pi}" upper="${177/180*pi}" effort="100" velocity="1" />
     <dynamics damping="0.2" friction="0" />
   </joint>
@@ -261,5 +261,5 @@
     <origin xyz="0 0 0.317" rpy="0 0 0 "/>
     <axis   xyz="0 1 0"/>
-    <limit lower="${-94/180*M_PI}" upper="${+94/180*M_PI}" effort="100" velocity="1" />
+    <limit lower="${-94/180*pi}" upper="${+94/180*pi}" effort="100" velocity="1" />
     <dynamics damping="0.2" friction="0" />
   </joint>
@@ -278,5 +278,5 @@
     <origin xyz="0 0 0" rpy="0 0 0 "/>
     <axis   xyz="0 0 1"/>
-    <limit lower="${-174/180*M_PI}" upper="${174/180*M_PI}" effort="100" velocity="2" />
+    <limit lower="${-174/180*pi}" upper="${174/180*pi}" effort="100" velocity="2" />
     <dynamics damping="0.2" friction="0" />
   </joint>
@@ -295,5 +295,5 @@
     <origin xyz="0 0 0.45" rpy="0 0 0 "/>
     <axis   xyz="0 1 0"/>
-    <limit lower="${-137/180*M_PI}" upper="${137/180*M_PI}" effort="100" velocity="2" />
+    <limit lower="${-137/180*pi}" upper="${137/180*pi}" effort="100" velocity="2" />
     <dynamics damping="0.2" friction="0" />
   </joint>
@@ -312,5 +312,5 @@
     <origin xyz="0 0 0" rpy="0 0 0 "/>
     <axis   xyz="0 0 1"/>
-    <limit lower="${-255/180*M_PI}" upper="${255/180*M_PI}" effort="100" velocity="6.28" />
+    <limit lower="${-255/180*pi}" upper="${255/180*pi}" effort="100" velocity="6.28" />
     <dynamics damping="0.2" friction="0" />
   </joint>
@@ -329,5 +329,5 @@
     <origin xyz="0 0 0.480" rpy="0 0 0 "/>
     <axis   xyz="0 1 0"/>
-    <limit lower="${-165/180*M_PI}" upper="${165/180*M_PI}" effort="100" velocity="6.28" />
+    <limit lower="${-165/180*pi}" upper="${165/180*pi}" effort="100" velocity="6.28" />
     <dynamics damping="0.2" friction="0" />
   </joint>
@@ -347,5 +347,5 @@
     <origin xyz="0 0 0.07" rpy="0 0 0 "/>
     <axis   xyz="0 0 1"/>
-    <limit lower="${-255/180*M_PI}" upper="${255/180*M_PI}" effort="100" velocity="6.28" />
+    <limit lower="${-255/180*pi}" upper="${255/180*pi}" effort="100" velocity="6.28" />
     <dynamics damping="0.2" friction="0" />
   </joint>

Commit message: use yaml robots file
- helpers.urdf.xacro: generic macros arm(), tool(), arm_with_tool()
- calibration files use scheme <tool name>_cal.xml or <arm name>_cal.xml
  where <tool name> and <arm name> match the names in the yaml settings file
- renamed link "*arm_hand_mount" to more generic "*tool_mount"

File: pa10-a.urdf.xacro (robot description, xacro)
@@ -361,8 +361,8 @@
   <joint name="${name}arm_hand_fixed_joint" type="fixed">
 	 <parent link="${name}arm_7_link"/>
-	 <child link="${name}arm_hand_mount"/>
-  </joint>
-  <link name="${name}arm_hand_mount" />
-  <gazebo reference="${name}arm_hand_mount">
+	 <child link="${name}tool_mount"/>
+  </joint>
+  <link name="${name}tool_mount" />
+  <gazebo reference="${name}tool_mount">
     <kinematic>${kinematic}</kinematic>
   </gazebo>

File: pa10-c.urdf.xacro (robot description, xacro)
@@ -361,8 +361,8 @@
   <joint name="${name}arm_hand_fixed_joint" type="fixed">
 	 <parent link="${name}arm_7_link"/>
-	 <child link="${name}arm_hand_mount"/>
-  </joint>
-  <link name="${name}arm_hand_mount" />
-   <gazebo reference="${name}arm_hand_mount">
+	 <child link="${name}tool_mount"/>
+  </joint>
+  <link name="${name}tool_mount" />
+   <gazebo reference="${name}tool_mount">
     <kinematic>${kinematic}</kinematic>
   </gazebo>
