Commit message: Moved pa10 description in its own package Restructured the package to match standard description package layouts

File: urdf/pa10-a.urdf.xacro (robot description, xacro)
@@ -5,5 +5,4 @@
 		 xmlns:controller="http://playerstage.sourceforge.net/gazebo/xmlschema/#controller"
        xmlns:interface="http://playerstage.sourceforge.net/gazebo/xmlschema/#interface">
-  <xacro:include filename="../urdf/util.urdf.xacro"/>
   <xacro:macro name="pa10a_arm" params="name kinematic:=false">
   <link name="${name}arm_base_link">
@@ -11,5 +10,5 @@
       <origin xyz="0 0 0" rpy="0 0 0"/>
       <geometry>
-        <mesh filename="package://agni_description/pa10/meshes/pa-7a/link0_mesh.dae" scale="1 1 1" />
+        <mesh filename="package://pa10_7a_description/meshes/pa-7a/link0_mesh.dae" scale="1 1 1" />
       </geometry>
     </visual>
@@ -41,5 +40,5 @@
       <origin xyz="0 0 0" rpy="0 0 0"/>
       <geometry>
-        <mesh filename="package://agni_description/pa10/meshes/pa-7a/link1_mesh.dae" scale="1 1 1" />
+        <mesh filename="package://pa10_7a_description/meshes/pa-7a/link1_mesh.dae" scale="1 1 1" />
       </geometry>
     </visual>
@@ -75,5 +74,5 @@
       <origin xyz="0 0 -0.315" rpy="0 0 3.1415"/>
       <geometry>
-        <mesh filename="package://agni_description/pa10/meshes/pa-7a/link2_mesh.dae" scale="1 1 1" />
+        <mesh filename="package://pa10_7a_description/meshes/pa-7a/link2_mesh.dae" scale="1 1 1" />
       </geometry>
     </visual>
@@ -103,5 +102,5 @@
       <origin xyz="0 0 -0.315" rpy="0 0 0"/>
       <geometry>
-        <mesh filename="package://agni_description/pa10/meshes/pa-7a/link3_mesh.dae" scale="1 1 1" />
+        <mesh filename="package://pa10_7a_description/meshes/pa-7a/link3_mesh.dae" scale="1 1 1" />
       </geometry>
     </visual>
@@ -137,5 +136,5 @@
       <origin xyz="0 0 -0.765" rpy="0 0 0"/>
       <geometry>
-        <mesh filename="package://agni_description/pa10/meshes/pa-7a/link4_mesh.dae" scale="1 1 1" />
+        <mesh filename="package://pa10_7a_description/meshes/pa-7a/link4_mesh.dae" scale="1 1 1" />
       </geometry>
     </visual>
@@ -165,5 +164,5 @@
       <origin xyz="0 0 -0.765" rpy="0 0 0"/>
       <geometry>
-        <mesh filename="package://agni_description/pa10/meshes/pa-7a/link5_mesh.dae" scale="1 1 1" />
+        <mesh filename="package://pa10_7a_description/meshes/pa-7a/link5_mesh.dae" scale="1 1 1" />
       </geometry>
     </visual>
@@ -199,5 +198,5 @@
       <origin xyz="0 0 -1.265" rpy="0 0 0"/>
       <geometry>
-        <mesh filename="package://agni_description/pa10/meshes/pa-7a/link6_mesh.dae" scale="1 1 1" />
+        <mesh filename="package://pa10_7a_description/meshes/pa-7a/link6_mesh.dae" scale="1 1 1" />
       </geometry>
     </visual>
@@ -221,5 +220,5 @@
       <origin xyz="0 0 1.345" rpy="0 0 0"/>
       <geometry>
-        <mesh filename="package://agni_description/pa10/meshes/pa-7a/link7_mesh.dae" scale="1 1 1" />
+        <mesh filename="package://pa10_7a_description/meshes/pa-7a/link7_mesh.dae" scale="1 1 1" />
       </geometry>
     </visual>

File: urdf/pa10-c.urdf.xacro (robot description, xacro)
@@ -11,5 +11,5 @@
       <origin xyz="0 0 0" rpy="0 0 0"/>
       <geometry>
-        <mesh filename="package://agni_description/pa10/meshes/pa-7c/link0_mesh.dae" scale="1 1 1" />
+        <mesh filename="package://pa10_7a_description/meshes/pa-7c/link0_mesh.dae" scale="1 1 1" />
       </geometry>
     </visual>
@@ -41,5 +41,5 @@
       <origin xyz="0 0 0" rpy="0 0 0"/>
       <geometry>
-        <mesh filename="package://agni_description/pa10/meshes/pa-7c/link1_mesh.dae" scale="1 1 1" />
+        <mesh filename="package://pa10_7a_description/meshes/pa-7c/link1_mesh.dae" scale="1 1 1" />
       </geometry>
     </visual>
@@ -75,5 +75,5 @@
       <origin xyz="0 0 -0.317" rpy="0 0 0"/>
       <geometry>
-        <mesh filename="package://agni_description/pa10/meshes/pa-7c/link2_mesh.dae" scale="1 1 1" />
+        <mesh filename="package://pa10_7a_description/meshes/pa-7c/link2_mesh.dae" scale="1 1 1" />
       </geometry>
     </visual>
@@ -103,5 +103,5 @@
       <origin xyz="0 0 -0.317" rpy="0 0 0"/>
       <geometry>
-        <mesh filename="package://agni_description/pa10/meshes/pa-7c/link3_mesh.dae" scale="1 1 1" />
+        <mesh filename="package://pa10_7a_description/meshes/pa-7c/link3_mesh.dae" scale="1 1 1" />
       </geometry>
     </visual>
@@ -137,5 +137,5 @@
       <origin xyz="0 0 -0.767" rpy="0 0 0"/>
       <geometry>
-        <mesh filename="package://agni_description/pa10/meshes/pa-7c/link4_mesh.dae" scale="1 1 1" />
+        <mesh filename="package://pa10_7a_description/meshes/pa-7c/link4_mesh.dae" scale="1 1 1" />
       </geometry>
     </visual>
@@ -165,5 +165,5 @@
       <origin xyz="0 0 -0.767" rpy="0 0 0"/>
       <geometry>
-        <mesh filename="package://agni_description/pa10/meshes/pa-7c/link5_mesh.dae" scale="1 1 1" />
+        <mesh filename="package://pa10_7a_description/meshes/pa-7c/link5_mesh.dae" scale="1 1 1" />
       </geometry>
     </visual>
@@ -199,5 +199,5 @@
       <origin xyz="0 0 -1.247" rpy="0 0 0"/>
       <geometry>
-        <mesh filename="package://agni_description/pa10/meshes/pa-7c/link6_mesh.dae" scale="1 1 1" />
+        <mesh filename="package://pa10_7a_description/meshes/pa-7c/link6_mesh.dae" scale="1 1 1" />
       </geometry>
     </visual>
@@ -221,5 +221,5 @@
       <origin xyz="0 0 0" rpy="0 0 0"/>
       <geometry>
-        <mesh filename="package://agni_description/pa10/meshes/pa-7c/link7_mesh.dae" scale="1 1 1" />
+        <mesh filename="package://pa10_7a_description/meshes/pa-7c/link7_mesh.dae" scale="1 1 1" />
       </geometry>
     </visual>

Commit message: Forked to create independent version 7c

File: urdf/pa10-a.urdf.xacro (robot description, xacro)
@@ -10,5 +10,5 @@
       <origin xyz="0 0 0" rpy="0 0 0"/>
       <geometry>
-        <mesh filename="package://pa10_7a_description/meshes/pa-7a/link0_mesh.dae" scale="1 1 1" />
+        <mesh filename="package://pa10_7c_description/meshes/pa-7a/link0_mesh.dae" scale="1 1 1" />
       </geometry>
     </visual>
@@ -40,5 +40,5 @@
       <origin xyz="0 0 0" rpy="0 0 0"/>
       <geometry>
-        <mesh filename="package://pa10_7a_description/meshes/pa-7a/link1_mesh.dae" scale="1 1 1" />
+        <mesh filename="package://pa10_7c_description/meshes/pa-7a/link1_mesh.dae" scale="1 1 1" />
       </geometry>
     </visual>
@@ -74,5 +74,5 @@
       <origin xyz="0 0 -0.315" rpy="0 0 3.1415"/>
       <geometry>
-        <mesh filename="package://pa10_7a_description/meshes/pa-7a/link2_mesh.dae" scale="1 1 1" />
+        <mesh filename="package://pa10_7c_description/meshes/pa-7a/link2_mesh.dae" scale="1 1 1" />
       </geometry>
     </visual>
@@ -102,5 +102,5 @@
       <origin xyz="0 0 -0.315" rpy="0 0 0"/>
       <geometry>
-        <mesh filename="package://pa10_7a_description/meshes/pa-7a/link3_mesh.dae" scale="1 1 1" />
+        <mesh filename="package://pa10_7c_description/meshes/pa-7a/link3_mesh.dae" scale="1 1 1" />
       </geometry>
     </visual>
@@ -136,5 +136,5 @@
       <origin xyz="0 0 -0.765" rpy="0 0 0"/>
       <geometry>
-        <mesh filename="package://pa10_7a_description/meshes/pa-7a/link4_mesh.dae" scale="1 1 1" />
+        <mesh filename="package://pa10_7c_description/meshes/pa-7a/link4_mesh.dae" scale="1 1 1" />
       </geometry>
     </visual>
@@ -164,5 +164,5 @@
       <origin xyz="0 0 -0.765" rpy="0 0 0"/>
       <geometry>
-        <mesh filename="package://pa10_7a_description/meshes/pa-7a/link5_mesh.dae" scale="1 1 1" />
+        <mesh filename="package://pa10_7c_description/meshes/pa-7a/link5_mesh.dae" scale="1 1 1" />
       </geometry>
     </visual>
@@ -198,5 +198,5 @@
       <origin xyz="0 0 -1.265" rpy="0 0 0"/>
       <geometry>
-        <mesh filename="package://pa10_7a_description/meshes/pa-7a/link6_mesh.dae" scale="1 1 1" />
+        <mesh filename="package://pa10_7c_description/meshes/pa-7a/link6_mesh.dae" scale="1 1 1" />
       </geometry>
     </visual>
@@ -220,5 +220,5 @@
       <origin xyz="0 0 1.345" rpy="0 0 0"/>
       <geometry>
-        <mesh filename="package://pa10_7a_description/meshes/pa-7a/link7_mesh.dae" scale="1 1 1" />
+        <mesh filename="package://pa10_7c_description/meshes/pa-7a/link7_mesh.dae" scale="1 1 1" />
       </geometry>
     </visual>

File: urdf/pa10-c.urdf.xacro (robot description, xacro)
@@ -11,5 +11,5 @@
       <origin xyz="0 0 0" rpy="0 0 0"/>
       <geometry>
-        <mesh filename="package://pa10_7a_description/meshes/pa-7c/link0_mesh.dae" scale="1 1 1" />
+        <mesh filename="package://pa10_7c_description/meshes/pa-7c/link0_mesh.dae" scale="1 1 1" />
       </geometry>
     </visual>
@@ -41,5 +41,5 @@
       <origin xyz="0 0 0" rpy="0 0 0"/>
       <geometry>
-        <mesh filename="package://pa10_7a_description/meshes/pa-7c/link1_mesh.dae" scale="1 1 1" />
+        <mesh filename="package://pa10_7c_description/meshes/pa-7c/link1_mesh.dae" scale="1 1 1" />
       </geometry>
     </visual>
@@ -75,5 +75,5 @@
       <origin xyz="0 0 -0.317" rpy="0 0 0"/>
       <geometry>
-        <mesh filename="package://pa10_7a_description/meshes/pa-7c/link2_mesh.dae" scale="1 1 1" />
+        <mesh filename="package://pa10_7c_description/meshes/pa-7c/link2_mesh.dae" scale="1 1 1" />
       </geometry>
     </visual>
@@ -103,5 +103,5 @@
       <origin xyz="0 0 -0.317" rpy="0 0 0"/>
       <geometry>
-        <mesh filename="package://pa10_7a_description/meshes/pa-7c/link3_mesh.dae" scale="1 1 1" />
+        <mesh filename="package://pa10_7c_description/meshes/pa-7c/link3_mesh.dae" scale="1 1 1" />
       </geometry>
     </visual>
@@ -137,5 +137,5 @@
       <origin xyz="0 0 -0.767" rpy="0 0 0"/>
       <geometry>
-        <mesh filename="package://pa10_7a_description/meshes/pa-7c/link4_mesh.dae" scale="1 1 1" />
+        <mesh filename="package://pa10_7c_description/meshes/pa-7c/link4_mesh.dae" scale="1 1 1" />
       </geometry>
     </visual>
@@ -165,5 +165,5 @@
       <origin xyz="0 0 -0.767" rpy="0 0 0"/>
       <geometry>
-        <mesh filename="package://pa10_7a_description/meshes/pa-7c/link5_mesh.dae" scale="1 1 1" />
+        <mesh filename="package://pa10_7c_description/meshes/pa-7c/link5_mesh.dae" scale="1 1 1" />
       </geometry>
     </visual>
@@ -199,5 +199,5 @@
       <origin xyz="0 0 -1.247" rpy="0 0 0"/>
       <geometry>
-        <mesh filename="package://pa10_7a_description/meshes/pa-7c/link6_mesh.dae" scale="1 1 1" />
+        <mesh filename="package://pa10_7c_description/meshes/pa-7c/link6_mesh.dae" scale="1 1 1" />
       </geometry>
     </visual>
@@ -221,5 +221,5 @@
       <origin xyz="0 0 0" rpy="0 0 0"/>
       <geometry>
-        <mesh filename="package://pa10_7a_description/meshes/pa-7c/link7_mesh.dae" scale="1 1 1" />
+        <mesh filename="package://pa10_7c_description/meshes/pa-7c/link7_mesh.dae" scale="1 1 1" />
       </geometry>
     </visual>
